File: hw/v3/ETH-IO_v3.1.brd (EAGLE design)
At the start: 100 x 85.4 mm, 82 parts, among them CON1 MC1,5-12-G-3,81, CON2 MC1,5-12-G-3,81, CON3 MC1,5-12-G-3,81, CON4 MC1,5-12-G-3,81, IC1 AP63205, IC2 TLP290-4, IC3 TLP290-4, IC4 TLP290-4, IC5 TLP290-4, IC6 TLP290-4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

Commit message: bigger footprints
Parts:
- removed L1: VLS5045EX-6R8M, my-inductor:L5040
- added JP1: (no value), pinhead:1X02
- added L3: VLS5045EX-6R8M, my-inductor:L5040-LONGER
- moved C9 2.61 mm to (22.4, 58.5), turned to 90 degrees
- moved C3 0.72 mm to (20.1, 58.5), turned to 90 degrees
Connections:
- net +24V: now also JP1.1
- net +5V: now also L3.1; no longer L1.1
- net GND: now also JP1.2
- net N$67: now also L3.2; no longer L1.2
Routing:
- net +24V: track 190.9 -> 196.6 mm
- net +5V: track 179.2 -> 182.8 mm
- net GND: track 13.0 -> 12.2 mm
- net C_S0-IN3: track 9.24 -> 8.68 mm
Other:
- board text added: "+"
- board text added: "-"
- board text added: "SJ"
